Commit message: - now compiles and run

File: src/my_robot_description/urdf/cubic_doggo.urdf.xacro (robot description, xacro)
@@ -30,5 +30,5 @@
         <visual>
             <geometry>
-                <mesh filename="package://my_robot_description/mesh/CADv0.1/basePlate.stl" scale="0.001 0.001 0.001"/>
+                <mesh filename="package://my_robot_description/mesh/CADv1/basePlate.stl" scale="0.001 0.001 0.001"/>
             </geometry>
             <origin xyz="0 0 0" rpy="0 0 0"/>
@@ -51,5 +51,5 @@
         <visual>
             <geometry>
-                <mesh filename="package://my_robot_description/mesh/CADv0.1/basePlate.stl" scale="0.001 0.001 0.001"/>
+                <mesh filename="package://my_robot_description/mesh/CADv1/basePlate.stl" scale="0.001 0.001 0.001"/>
             </geometry>
             <origin xyz="0 0 0" rpy="0 0 0"/>

File: src/my_robot_description/urdf/cubic_doggo_leg.xacro (robot description, xacro)
@@ -30,5 +30,5 @@
         <visual>
             <geometry>
-                <mesh filename="package://my_robot_description/mesh/CADv0.1/XL430holderBasic.stl" scale="0.001 0.001 0.001"/>
+                <mesh filename="package://my_robot_description/mesh/CADv1/XL430holderBasic.stl" scale="0.001 0.001 0.001"/>
             </geometry>
             <material name="white"/>
@@ -97,5 +97,5 @@
         <visual>
             <geometry>
-                <mesh filename="package://my_robot_description/mesh/CADv0.1/XL430holderBasic.stl" scale="0.001 0.001 0.001"/>
+                <mesh filename="package://my_robot_description/mesh/CADv1/XL430holderBasic.stl" scale="0.001 0.001 0.001"/>
             </geometry>
             <material name="white"/>
@@ -165,5 +165,5 @@
         <visual>
             <geometry>
-                <mesh filename="package://my_robot_description/mesh/CADv0.1/thighInner.stl" scale="0.001 0.001 0.001"/>
+                <mesh filename="package://my_robot_description/mesh/CADv1/thighInner.stl" scale="0.001 0.001 0.001"/>
             </geometry>
             <material name="blue"/>
@@ -187,5 +187,5 @@
         <visual>
             <geometry>
-                <mesh filename="package://my_robot_description/mesh/CADv0.1/thighOuter.stl" scale="0.001 0.001 0.001"/>
+                <mesh filename="package://my_robot_description/mesh/CADv1/thighOuter.stl" scale="0.001 0.001 0.001"/>
             </geometry>
             <material name="blue"/>
@@ -231,5 +231,5 @@
         <visual>
             <geometry>
-                <mesh filename="package://my_robot_description/mesh/CADv0.1/calfFeet.stl" scale="0.001 0.001 0.001"/>
+                <mesh filename="package://my_robot_description/mesh/CADv1/calfFeet.stl" scale="0.001 0.001 0.001"/>
             </geometry>
             <material name="purple"/>
@@ -256,5 +256,5 @@
         <visual>
             <geometry>
-                <mesh filename="package://my_robot_description/mesh/CADv0.1/calfJoint.stl" scale="0.001 0.001 0.001"/>
+                <mesh filename="package://my_robot_description/mesh/CADv1/calfJoint.stl" scale="0.001 0.001 0.001"/>
             </geometry>
             <origin xyz="0 0 0" rpy="${urdf_pi/2} 0 ${-rflc*urdf_pi/2}"/>
